Commit message: added hybrid astar, added interface of action btn gym and MPC_controller

File: obstacled_environments/common/plane_small.urdf (robot description, URDF)
Before this commit: robot plane, 1 links, 0 joints
Links:
- link planeLink: geometry collision box size=800 800 10; visual mesh filename=meshes/plane_small.obj scale=1 1 1
